Commit message: add virtual link for global referance for help navigation

File: my_robot.urdf (robot description, URDF)
Before this commit: robot kavee, 5 links, 4 joints
Links:
- added link base_footprint
Joints:
- added joint base_joint: type fixed, parent base_footprint, child base_link, origin xyz=0 0 0.1 rpy=0 0 0
