Commit message: add turtle bot wheels stl and add gazebo launch file

File: my_custom_robot/urdf/my_robot.urdf (robot description, URDF)
Before this commit: robot kavee, 6 links, 5 joints
Links:
- link base_footprint: mass None -> 0.1
- link base_link: mass None -> 15.0; geometry collision box size=0.6 0.4 0.2; visual box size=0.6 0.4 0.2
- link caster_link: mass None -> 1.0; geometry collision sphere radius=0.0825; visual sphere radius=0.0825
- link left_wheel_link: mass None -> 2.0; geometry collision cylinder length=0.091 radius=0.165; visual mesh filename=package://my_custom_robot/meshes/left_tire.stl scale=0.005 0.005 0.005
- link lidar_link: mass None -> 0.5; geometry collision cylinder length=0.05 radius=0.1; visual cylinder length=0.05 radius=0.1
- link right_wheel_link: mass None -> 2.0; geometry collision cylinder length=0.091 radius=0.165; visual mesh filename=package://my_custom_robot/meshes/right_tire.stl scale=0.005 0.005 0.005
Joints:
- joint base_caster_joint: origin xyz=0.2 0 -0.05 rpy=0 0 0 -> xyz=0.2 0 -0.0825 rpy=0 0 0
- joint base_joint: origin xyz=0 0 0.1 rpy=0 0 0 -> xyz=0 0 0.165 rpy=0 0 0
- joint base_left_wheel_joint: origin xyz=-0.15 0.225 0 rpy=0 0 0 -> xyz=-0.15 0.250 0 rpy=0 0 0
- joint base_right_wheel_joint: origin xyz=-0.15 -0.225 0 rpy=0 0 0 -> xyz=-0.15 -0.250 0 rpy=0 0 0

Commit message: added lidar from turtlebot3 waffel pi and make it responsive

File: my_custom_robot/urdf/my_robot.urdf (robot description, URDF)
Before this commit: robot kavee, 6 links, 5 joints
Links:
- link lidar_link: geometry collision cylinder length=0.05 radius=0.1; visual mesh filename=package://my_custom_robot/meshes/lds.stl scale=0.005 0.005 0.005
